Commit message: Fix measurement inconsistencies found during handover audit
- v3 firmware: wheel separation 0.47m → 0.44m (physically verified)
- URDF: laser_frame height 0.23m → 0.22m (physically measured)
- rplidar_with_transform: laser Z offset 0.20m → 0.22m (matches URDF)
- README: confirm encoder 1000 PPR / 4000 CPR, add map generation note

Co-Authored-By: Claude Sonnet 4.6 <noreply@anthropic.com>

File: ros2_ws/src/rover_description/urdf/rover.urdf (robot description, URDF)
Before this commit: robot expo_rover, 5 links, 4 joints
Joints:
- joint laser_joint: origin xyz=0.0 0.0 0.23 rpy=0 0 0 -> xyz=0.0 0.0 0.22 rpy=0 0 0

Commit message: Add RealSense D455 support, command reference, and robot front-marker
- realsense.launch.py: bring up the D455 for the rover (depth, color,
  aligned depth, NEON pointcloud) + base_link->camera_link mount TF.
  IMU disabled (RSUSB backend can't reach the HID motion sensor);
  initial_reset off (caused USB-2 re-enumerate churn). Camera confirmed
  publishing /camera/camera/depth/color/points on the AGX Orin.
- COMMANDS.md: full startup/operations reference for the whole rover
  (SLAM bringup, teleop, firmware flashing, health checks, wiring, calib).
- rover.urdf: bright green front-marker so the robot's forward direction
  is unambiguous in the viewer (chassis box was symmetric).
- .gitignore: ignore regenerable maps/ output.

Co-Authored-By: Claude Opus 4.8 <noreply@anthropic.com>

File: ros2_ws/src/rover_description/urdf/rover.urdf (robot description, URDF)
Before this commit: robot expo_rover, 5 links, 4 joints
Links:
- link base_link: geometry collision box size=0.43 0.44 0.23; visual box size=0.06 0.14 0.08
